File: dip28/dip28.kicad_sch (KiCad schematic)
At the start: 8 parts, among them J1 PinHeader_1x06_P2.54mm_Horizo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, U1 ATmega328-P, Y1 16MHz

Commit message: fixed pogo and dip adapter
Parts:
- U1: footprint Socket:DIP_Socket-28_W6.9_W7.62_W10.16_W12.7_W13.5_3M_228-4817-00-0602J -> (none)
Changed lines of the file:
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@@
       (effects (font (size 1.27 1.27)) (justify right))
     )
-    (property "Footprint" "Socket:DIP_Socket-28_W6.9_W7.62_W10.16_W12.7_W13.5_3M_228-4817-00-0602J" (id 2) (at 123.825 103.505 0)
+    (property "Footprint" "" (id 2) (at 123.825 103.505 0)
       (effects (font (size 1.27 1.27) italic) hide)
     )
@@
     )
     (path "/0c96e642-b7e3-494e-a132-98e02e803b47"
-      (reference "U1") (unit 1) (value "ATmega328-P") (footprint "Socket:DIP_Socket-28_W6.9_W7.62_W10.16_W12.7_W13.5_3M_228-4817-00-0602J")
+      (reference "U1") (unit 1) (value "ATmega328-P") (footprint "Socket:DIP_Socket-28_W11.9_W12.7_W15.24_W17.78_W18.5_3M_228-1277-00-0602J")
     )
     (path "/74fd1e5e-eaed-44c7-b443-9c8aaba887bc"
